File: CAN_PMOD/CAN_PMOD.kicad_sch (KiCad schematic)
At the start: 1 part, among them J1 Generic Conn 02x06 Horizontal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

Commit message: Work in schematic
Parts:
- added C? (x2): 100pF, Capacitor_SMD:C_0603_1608Metric, symbol Device:C
- added D?: NUP2105L, Package_TO_SOT_SMD:SOT-23, symbol Power_Protection:NUP2105L
- added J? (x2): Conn_01x03, Connector_PinHeader_2.54mm:PinHeader_1x03_P2.54mm_Vertical, symbol Connector_Generic:Conn_01x03
- added J? (x3): TH 01x02 2.54mm, Connector_PinHeader_2.54mm:PinHeader_1x02_P2.54mm_Vertical, symbol Connector_Generic:Conn_01x02
- added J?: DB9_Female_MountingHoles, symbol Connector:DB9_Female_MountingHoles
- added R? (x2): 120, Resistor_SMD:R_0603_1608Metric, symbol Device:R
- added R?: 0, Resistor_SMD:R_0603_1608Metric, symbol Device:R
- added U?: CAN Transceiver, Package_SO:SOIC-8_3.9x4.9mm_P1.27mm, symbol symbol_lib:CAN Transceiver
- added U?: MCP2515-xSO, Package_SO:SOIC-18W_7.5x11.6mm_P1.27mm, symbol Interface_CAN_LIN:MCP2515-xSO
- J1: value Generic Conn 02x06 Horizontal 2.54mm pitch -> TH 02x06 Horizontal 2.54mm
Connections:
- net +3V3: now also C?.1, U?.18 (VDD), U?.3 (VCC)
- net CAN_RX: now also J?.2 (Pin_2), U?.4 (RX); no longer J1.7 (Pin_7)
- net CAN_TX: now also J?.2 (Pin_2), U?.1 (TXD); no longer J1.8 (Pin_8)
- net GND: now also C?.2, C?.2, D?.3 (A), J?.2 (Pin_2), U?.2 (GND), U?.9 (VSS)
- net SPI_CS: now also U?.16 (~{CS})
- net SPI_MISO: now also U?.15 (SO)
- net SPI_MOSI: now also U?.14 (SI)
- net SPI_SCK: now also U?.13 (SCK)
- net GPIO renamed #RST
- net #RST: now also U?.17 (~{RESET})
- net INT renamed #INT
- net #INT: now also U?.12 (~{INT})
- new net: J?.2 (Pin_2), R?.1 (x2)
- new net: C?.1, R?.2, R?.2
- new net: J?.1 (Pin_1), R?.1
- new net: R?.2, U?.8 (S/NC)
- new net CAN_N: D?.2 (K), J?.1 (Pin_1), U?.6 (CAN_L)
- new net CAN_P: D?.1 (K), J?.1 (Pin_1), U?.7 (CAN_H)
- new net CAN_RX_IN: J1.7 (Pin_7), J?.1 (Pin_1)
- new net CAN_TX_IN: J1.8 (Pin_8), J?.1 (Pin_1)
- new net RX_CAN: J?.3 (Pin_3), U?.2 (RXCAN)
- new net TX_CAN: J?.3 (Pin_3), U?.1 (TXCAN)
- no-connect marks 0 -> 1
Other:
- note added: "Component Notes: ============ - Default C: 0603 16v 10% X7R - Default R: 0603 75v 5%"
- note added: "Design objectives: =========== - Cheap - Multi part number design for stock problems - Optional use of SPI to CAN TX/RX converter - Option to enable previous using jumpers"
- note added: "For those PN selecting speed, connect the jumper for high-speed mode"
- note added: "If desited, change value for slope-control PNs"
- note added: "Layout Notes: ========= - Follow PMOD v1.3 Standard for dimensions and connector clearance"
- note added: "Layout: place near connector"
- note added: "Part Number | Pin 5 | Pin 8 -------------------- SN65HVD232D NC NC SN65HVD230D VREF RS SN65HVD231D VREF RS TCAN330D SHDN Silent TCAN332D NC NC TCAN334D SHDN STB TCAN330D FAULT Silent SN65HVD233D LBK RS SN65HVD230D VREF RS"
- note added: "REVIEW COMPONENT"
- note removed: "Design objectives: - CAN transceiver with standard footprint and pinout for part number switching - Optional use of SPI to CAN TX/RX converter - Option to enable previous using jumpers"
- moved on the sheet: J1
